Commit message: Created ROS2 package

File: manipulator_gazebo/model/manipulator/manipulator.urdf (robot description, URDF)
Before this commit: robot manipulator, 5 links, 4 joints
Links:
- link base_link: geometry collision mesh filename=/home/ekumen/colcon_ws/src/manipulator_sim/manipulator_gaze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; visual mesh filename=/home/ekumen/colcon_ws/src/manipulator_sim/manipulator_gaze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
- link link_1: geometry collision mesh filename=/home/ekumen/colcon_ws/src/manipulator_sim/manipulator_gaze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; visual mesh filename=/home/ekumen/colcon_ws/src/manipulator_sim/manipulator_gaze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
- link link_2: geometry collision mesh filename=/home/ekumen/colcon_ws/src/manipulator_sim/manipulator_gaze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; visual mesh filename=/home/ekumen/colcon_ws/src/manipulator_sim/manipulator_gaze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
- link link_3: geometry collision mesh filename=/home/ekumen/colcon_ws/src/manipulator_sim/manipulator_gaze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; visual mesh filename=/home/ekumen/colcon_ws/src/manipulator_sim/manipulator_gaze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

File: manipulator_gazebo/urdf/manipulator.urdf.xacro (robot description, xacro)
@@ -27,5 +27,5 @@
         <origin xyz="0 0 0" rpy="0 0 0" />
         <geometry>
-          <mesh filename="$(cwd)/model/manipulator/base.stl"/>
+          <mesh filename="$(cwd)/manipulator_gazebo/model/manipulator/base.stl"/>
         </geometry>
       </visual>
@@ -33,5 +33,5 @@
         <origin xyz="0 0 0" rpy="0 0 0" />
         <geometry>
-          <mesh filename="$(cwd)/model/manipulator/base.stl"/>
+          <mesh filename="$(cwd)/manipulator_gazebo/model/manipulator/base.stl"/>
         </geometry>
       </collision>
@@ -51,5 +51,5 @@
         <origin xyz="0 0 0" rpy="0 0 0" />
         <geometry>
-          <mesh filename="$(cwd)/model/manipulator/link_1.stl"/>
+          <mesh filename="$(cwd)/manipulator_gazebo/model/manipulator/link_1.stl"/>
         </geometry>
       </visual>
@@ -57,5 +57,5 @@
         <origin xyz="0 0 0" rpy="0 0 0" />
         <geometry>
-          <mesh filename="$(cwd)/model/manipulator/link_1.stl"/>
+          <mesh filename="$(cwd)/manipulator_gazebo/model/manipulator/link_1.stl"/>
         </geometry>
       </collision>
@@ -76,5 +76,5 @@
         <origin xyz="0 0 0" rpy="0 0 0" />
         <geometry>
-          <mesh filename="$(cwd)/model/manipulator/link_2.stl"/>
+          <mesh filename="$(cwd)/manipulator_gazebo/model/manipulator/link_2.stl"/>
         </geometry>
       </visual>
@@ -82,5 +82,5 @@
         <origin xyz="0 0 0" rpy="0 0 0" />
         <geometry>
-          <mesh filename="$(cwd)/model/manipulator/link_2.stl"/>
+          <mesh filename="$(cwd)/manipulator_gazebo/model/manipulator/link_2.stl"/>
         </geometry>
       </collision>
@@ -101,5 +101,5 @@
         <origin xyz="0 0 0" rpy="0 0 0" />
         <geometry>
-          <mesh filename="$(cwd)/model/manipulator/link_3.stl"/>
+          <mesh filename="$(cwd)/manipulator_gazebo/model/manipulator/link_3.stl"/>
         </geometry>
       </visual>
@@ -107,5 +107,5 @@
         <origin xyz="0 0 0" rpy="0 0 0" />
         <geometry>
-          <mesh filename="$(cwd)/model/manipulator/link_3.stl"/>
+          <mesh filename="$(cwd)/manipulator_gazebo/model/manipulator/link_3.stl"/>
         </geometry>
       </collision>

Commit message: Finally working

File: manipulator_gazebo/model/manipulator/manipulator.urdf (robot description, URDF)
Before this commit: robot manipulator, 5 links, 4 joints
Joints:
- joint joint_2: limit lower=0.7853981633974483 upper=1.5707963267948966 effort=1000.0 velocity=1.0 -> lower=0 upper=1.5707963267948966 effort=1000.0 velocity=1.0
- joint joint_3: limit lower=-3.141592653589793 upper=1.5707963267948966 effort=1000.0 velocity=1.0 -> lower=-3.141592653589793 upper=3.141592653589793 effort=1000.0 velocity=1.0; origin xyz=0.25 0 0 rpy=0 0 0 -> xyz=0.25 0 0 rpy=3.141592653589793 3.141592653589793 0

File: manipulator_gazebo/urdf/manipulator.urdf.xacro (robot description, xacro)
@@ -64,4 +64,5 @@
     <gazebo reference="link_1">
       <material>Gazebo/White</material>
+      <turnGravityOff>true</turnGravityOff>
     </gazebo>
     <joint name="joint_2" type="revolute">
@@ -69,5 +70,5 @@
       <child link="link_2"/>
       <axis xyz="0 0 1"/>
-      <limit effort="1000.0" lower="${pi/4}" upper="${pi/2}" velocity="1.0"/>
+      <limit effort="1000.0" lower="0" upper="${pi/2}" velocity="1.0"/>
       <origin xyz="0 0 ${link1_length}" rpy="${pi/2} 0 0"/>
     </joint>
@@ -89,4 +90,5 @@
     <gazebo reference="link_2">
       <material>Gazebo/Blue</material>
+      <turnGravityOff>true</turnGravityOff>
     </gazebo>
     <joint name="joint_3" type="revolute">
@@ -94,6 +96,6 @@
       <child link="link_3"/>
       <axis xyz="0 0 1"/>
-      <limit effort="1000.0" lower="${-pi}" upper="${pi/2}" velocity="1.0"/>
-      <origin xyz="${link2_length} 0 0" rpy="0 0 0"/>
+      <limit effort="1000.0" lower="${-pi}" upper="${pi}" velocity="1.0"/>
+      <origin xyz="${link2_length} 0 0" rpy="${pi} ${pi} 0"/>
     </joint>
     <link name="link_3">
@@ -114,4 +116,5 @@
     <gazebo reference="link_3">
       <material>Gazebo/Green</material>
+      <turnGravityOff>true</turnGravityOff>
     </gazebo>
     <gazebo>

Commit message: passing in arguments

File: manipulator_gazebo/model/manipulator/manipulator.urdf (robot description, URDF)
Before this commit: robot manipulator, 5 links, 4 joints
Links:
- link base_link: geometry collision mesh filename=/home/rodri/colcon_ws/src/manipulator_sim/manipulator_gazeb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; visual mesh filename=/home/rodri/colcon_ws/src/manipulator_sim/manipulator_gazeb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
- link link_1: geometry collision mesh filename=/home/rodri/colcon_ws/src/manipulator_sim/manipulator_gazeb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; visual mesh filename=/home/rodri/colcon_ws/src/manipulator_sim/manipulator_gazeb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
- link link_2: geometry collision mesh filename=/home/rodri/colcon_ws/src/manipulator_sim/manipulator_gazeb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; visual mesh filename=/home/rodri/colcon_ws/src/manipulator_sim/manipulator_gazeb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
- link link_3: geometry collision mesh filename=/home/rodri/colcon_ws/src/manipulator_sim/manipulator_gazeb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; visual mesh filename=/home/rodri/colcon_ws/src/manipulator_sim/manipulator_gazeb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

Commit message: prints pose of tool

File: manipulator_gazebo/model/manipulator/manipulator.urdf (robot description, URDF)
Before this commit: robot manipulator, 5 links, 4 joints
Links:
- added link link_4, mass 1.0; collision mesh filename=/home/rodri/colcon_ws/src/manipulator_sim/manipulator_gazeb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; visual mesh filename=/home/rodri/colcon_ws/src/manipulator_sim/manipulator_gazeb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
Joints:
- added joint joint_4: type fixed, parent link_3, child link_4, origin xyz=0.2 0 0 rpy=0 0 0

File: manipulator_gazebo/urdf/manipulator.urdf.xacro (robot description, xacro)
@@ -118,4 +118,30 @@
       <turnGravityOff>true</turnGravityOff>
     </gazebo>
+    <joint name="joint_4" type="fixed">
+      <parent link="link_3"/>
+      <child link="link_4"/>
+      <origin xyz="${link3_length} 0 0" rpy="0 0 0"/>
+    </joint>
+    <link name="link_4">
+      <visual>
+        <origin xyz="0 0 0" rpy="0 0 0" />
+        <geometry>
+          <mesh filename="$(cwd)/manipulator_gazebo/model/manipulator/sphere.stl"/>
+        </geometry>
+      </visual>
+      <collision>
+        <origin xyz="0 0 0" rpy="0 0 0" />
+        <geometry>
+          <mesh filename="$(cwd)/manipulator_gazebo/model/manipulator/sphere.stl"/>
+        </geometry>
+      </collision>
+      <xacro:inertial_dummy/>
+    </link>
+    <gazebo reference="joint_4">
+      <preserveFixedJoint>true</preserveFixedJoint>
+    </gazebo>
+    <gazebo reference="link_4">
+      <turnGravityOff>true</turnGravityOff>
+    </gazebo>
     <gazebo>
       <plugin name="manipulator_drive_plugin" filename="libmanipulator_drive.so">

Commit message: fixes bug in calculation of a3

File: manipulator_gazebo/model/manipulator/manipulator.urdf (robot description, URDF)
Before this commit: robot manipulator, 6 links, 5 joints
Joints:
- joint joint_2: limit lower=0 upper=1.5707963267948966 effort=1000.0 velocity=1.0 -> (none); type revolute -> continuous
- joint joint_3: limit lower=-3.141592653589793 upper=3.141592653589793 effort=1000.0 velocity=1.0 -> (none); type revolute -> continuous

File: manipulator_gazebo/urdf/manipulator.urdf.xacro (robot description, xacro)
@@ -66,9 +66,8 @@
       <turnGravityOff>true</turnGravityOff>
     </gazebo>
-    <joint name="joint_2" type="revolute">
+    <joint name="joint_2" type="continuous">
       <parent link="link_1"/>
       <child link="link_2"/>
       <axis xyz="0 0 1"/>
-      <limit effort="1000.0" lower="0" upper="${pi/2}" velocity="1.0"/>
       <origin xyz="0 0 ${link1_length}" rpy="${pi/2} 0 0"/>
     </joint>
@@ -92,9 +91,8 @@
       <turnGravityOff>true</turnGravityOff>
     </gazebo>
-    <joint name="joint_3" type="revolute">
+    <joint name="joint_3" type="continuous">
       <parent link="link_2"/>
       <child link="link_3"/>
       <axis xyz="0 0 1"/>
-      <limit effort="1000.0" lower="${-pi}" upper="${pi}" velocity="1.0"/>
       <origin xyz="${link2_length} 0 0" rpy="${pi} ${pi} 0"/>
     </joint>
